Commit message: Gazebo works and ros

File: install/my_robot_description/share/my_robot_description/urdf/camera.xacro (robot description, xacro)
@@ -29,5 +29,5 @@
     <origin xyz="${(base_length+camera_link_length) / 2.0} 0.0 ${base_height / 2.0}" rpy="0.0 0.0 0.0"/>
   </joint>
-  <!-- Optical frame -->
+  <!-- Optical frame for camera to emilate the real world blue light -->
   <link name="camera_optical_link"/>
   <joint name="camera_optical_joint" type="fixed">

File: install/my_robot_description/share/my_robot_description/urdf/common_properties.xacro (robot description, xacro)
@@ -6,4 +6,10 @@
     <material name="grey">
         <color rgba="0.5 0.5 0.5 1" />
+    </material>
+    <material name="orange">
+        <color rgba="1 0.5 0 1" />
+    </material>
+    <material name="yellow">
+        <color rgba="1 1 0 1" />
     </material>
     <xacro:macro name="box_inertia" params="m x y z o_xyz o_rpy">

File: install/my_robot_description/share/my_robot_description/urdf/my_robot.urdf.xacro (robot description, xacro)
@@ -5,3 +5,11 @@
     <xacro:include filename="mobile_base_gazebo.xacro" />
     <xacro:include filename="camera.xacro" />
+    <xacro:include filename="arm.xacro" />
+    <xacro:include filename="arm_base_gazebo.xacro" />
+    <!-- Define base dimensions -->
+    <joint name="arm_base_mobile_joint" type="fixed">
+        <origin xyz="0.2 0.0 0.2" rpy="0.0 0.0 0.0"/>
+        <parent link="base_link"/>
+        <child link="arm_base_link"/>
+    </joint>
 </robot>
